Commit message: picks good

File: src/planning/models/block/model.urdf (robot description, URDF)
Before this commit: robot block, 1 links, 0 joints
Links:
- link block: geometry collision box size=0.025 0.025 0.025; visual box size=0.025 0.025 0.025

File: src/planning/models/block/model2.urdf (robot description, URDF)
Before this commit: robot block2, 1 links, 0 joints
Links:
- link block2: geometry collision box size=0.025 0.025 0.025; visual box size=0.025 0.025 0.025
